Commit message: add arm controllers

File: lekiwi_description/urdf/LeKiwi_ros2_control.xacro (robot description, xacro)
@@ -15,4 +15,46 @@
             <plugin>gz_ros2_control/GazeboSimSystem</plugin>
         </hardware>
+        <joint name="STS3215_03a-v1_Revolute-45">
+                <command_interface name="position"/>
+                <state_interface name="position">
+                  <param name="initial_value">0</param>
+                </state_interface>
+                <state_interface name="velocity"/>
+            </joint>
+            <joint name="STS3215_03a-v1-1_Revolute-49">
+                <command_interface name="position"/>
+                <state_interface name="position">
+                  <param name="initial_value">0</param>
+                </state_interface>
+                <state_interface name="velocity"/>
+            </joint>
+            <joint name="STS3215_03a-v1-2_Revolute-51">
+                <command_interface name="position"/>
+                <state_interface name="position">
+                  <param name="initial_value">0</param>
+                </state_interface>
+                <state_interface name="velocity"/>
+            </joint>
+            <joint name="STS3215_03a-v1-3_Revolute-53">
+                <command_interface name="position"/>
+                <state_interface name="position">
+                  <param name="initial_value">0</param>
+                </state_interface>
+                <state_interface name="velocity"/>
+            </joint>
+            <joint name="STS3215_03a_Wrist_Roll-v1_Revolute-55">
+                <command_interface name="position"/>
+                <state_interface name="position">
+                  <param name="initial_value">0</param>
+                </state_interface>
+                <state_interface name="velocity"/>
+            </joint>
+            <joint name="STS3215_03a-v1-4_Revolute-57">
+                <command_interface name="position"/>
+                <state_interface name="position">
+                  <param name="initial_value">0</param>
+                </state_interface>
+                <state_interface name="velocity"/>
+            </joint>
         <xacro:wheel_control name="ST3215_Servo_Motor-v1-2_Revolute-60" />
         <xacro:wheel_control name="ST3215_Servo_Motor-v1-1_Revolute-62" />
