Commit message: add colors to links

File: lekiwi_description/urdf/LeKiwi.xacro (robot description, xacro)
@@ -3,4 +3,19 @@
     <xacro:include filename="$(find lekiwi_description)/urdf/LeKiwi_ros2_control.xacro" />
     <xacro:include filename="$(find lekiwi_description)/urdf/LeKiwi_gazebo.xacro" />
+    <!-- ===== MATERIAL DEFINITIONS ===== -->
+    <material name="base_dark_gray"><color rgba="0.25 0.25 0.25 1.0"/></material>
+    <material name="orange"><color rgba="0.95 0.5 0.1 1.0"/></material>
+    <material name="servo_gray"><color rgba="0.30 0.30 0.35 1.0"/></material>
+    <material name="wheel_mount_silver"><color rgba="0.70 0.70 0.72 1.0"/></material>
+    <material name="wheel_black"><color rgba="0.08 0.08 0.08 1.0"/></material>
+    <material name="light_gray"><color rgba="0.75 0.75 0.75 1.0"/></material>
+    <material name="battery_green"><color rgba="0.15 0.60 0.20 1.0"/></material>
+    <material name="silver"><color rgba="0.82 0.82 0.85 1.0"/></material>
+    <material name="arm_blue"><color rgba="0.18 0.38 0.72 1.0"/></material>
+    <material name="arm_blue_dark"><color rgba="0.12 0.25 0.55 1.0"/></material>
+    <material name="arm_servo"><color rgba="0.22 0.22 0.28 1.0"/></material>
+    <material name="gripper_teal"><color rgba="0.10 0.65 0.65 1.0"/></material>
+    <material name="cam_black"><color rgba="0.10 0.10 0.10 1.0"/></material>
+    <material name="pcb_green"><color rgba="0.12 0.45 0.18 1.0"/></material>
     <link name="base_footprint"/>
     <link name="base_plate_layer1-v5">
@@ -15,4 +30,5 @@
                 <mesh filename="package://lekiwi_description/meshes/base_plate_layer1-v5.stl" scale="0.001 0.001 0.001" />
             </geometry>
+            <material name="base_dark_gray"/>
         </visual>
         <collision name="base_plate_layer1-v5_collision">
@@ -34,4 +50,5 @@
                 <mesh filename="package://lekiwi_description/meshes/drive_motor_mount-v11-2.stl" scale="0.001 0.001 0.001" />
             </geometry>
+            <material name="orange"/>
         </visual>
         <collision name="drive_motor_mount-v11-2_collision">
@@ -53,4 +70,5 @@
                 <mesh filename="package://lekiwi_description/meshes/ST3215_Servo_Motor-v1-2.stl" scale="0.001 0.001 0.001" />
             </geometry>
+            <material name="servo_gray"/>
         </visual>
         <collision name="ST3215_Servo_Motor-v1-2_collision">
@@ -72,4 +90,5 @@
                 <mesh filename="package://lekiwi_description/meshes/4-Omni-Directional-Wheel_Single_Body-v1-2.stl" scale="0.001 0.001 0.001" />
             </geometry>
+            <material name="wheel_black"/>
         </visual>
         <collision name="4-Omni-Directional-Wheel_Single_Body-v1-2_collision">
@@ -91,4 +110,5 @@
                 <mesh filename="package://lekiwi_description/meshes/omni_wheel_mount-v5-2.stl" scale="0.001 0.001 0.001" />
             </geometry>
+            <material name="wheel_mount_silver"/>
         </visual>
         <collision name="omni_wheel_mount-v5-2_collision">
@@ -110,4 +130,5 @@
                 <mesh filename="package://lekiwi_description/meshes/drive_motor_mount-v11-1.stl" scale="0.001 0.001 0.001" />
             </geometry>
+            <material name="orange"/>
         </visual>
         <collision name="drive_motor_mount-v11-1_collision">
@@ -129,4 +150,5 @@
                 <mesh filename="package://lekiwi_description/meshes/ST3215_Servo_Motor-v1-1.stl" scale="0.001 0.001 0.001" />
             </geometry>
+            <material name="servo_gray"/>
         </visual>
         <collision name="ST3215_Servo_Motor-v1-1_collision">
@@ -148,4 +170,5 @@
                 <mesh filename="package://lekiwi_description/meshes/omni_wheel_mount-v5-1.stl" scale="0.001 0.001 0.001" />
             </geometry>
+            <material name="wheel_mount_silver"/>
         </visual>
         <collision name="omni_wheel_mount-v5-1_collision">
@@ -167,4 +190,5 @@
                 <mesh filename="package://lekiwi_description/meshes/4-Omni-Directional-Wheel_Single_Body-v1-1.stl" scale="0.001 0.001 0.001" />
             </geometry>
+            <material name="wheel_black"/>
         </visual>
         <collision name="4-Omni-Directional-Wheel_Single_Body-v1-1_collision">
@@ -186,4 +210,5 @@
                 <mesh filename="package://lekiwi_description/meshes/drive_motor_mount-v11.stl" scale="0.001 0.001 0.001" />
             </geometry>
+            <material name="orange"/>
         </visual>
         <collision name="drive_motor_mount-v11_collision">
@@ -205,4 +230,5 @@
                 <mesh filename="package://lekiwi_description/meshes/ST3215_Servo_Motor-v1.stl" scale="0.001 0.001 0.001" />
             </geometry>
+            <material name="servo_gray"/>
         </visual>
         <collision name="ST3215_Servo_Motor-v1_collision">
@@ -224,4 +250,5 @@
                 <mesh filename="package://lekiwi_description/meshes/omni_wheel_mount-v5.stl" scale="0.001 0.001 0.001" />
             </geometry>
+            <material name="wheel_mount_silver"/>
         </visual>
         <collision name="omni_wheel_mount-v5_collision">
@@ -243,4 +270,5 @@
                 <mesh filename="package://lekiwi_description/meshes/4-Omni-Directional-Wheel_Single_Body-v1.stl" scale="0.001 0.001 0.001" />
             </geometry>
+            <material name="wheel_black"/>
         </visual>
         <collision name="4-Omni-Directional-Wheel_Single_Body-v1_collision">
@@ -262,4 +290,5 @@
                 <mesh filename="package://lekiwi_description/meshes/servo_controller_mount-v3.stl" scale="0.001 0.001 0.001" />
             </geometry>
+            <material name="light_gray"/>
         </visual>
         <collision name="servo_controller_mount-v3_collision">
@@ -281,4 +310,5 @@
                 <mesh filename="package://lekiwi_description/meshes/lipo_battery_mount-v3.stl" scale="0.001 0.001 0.001" />
             </geometry>
+            <material name="light_gray"/>
         </visual>
         <collision name="lipo_battery_mount-v3_collision">
@@ -300,4 +330,5 @@
                 <mesh filename="package://lekiwi_description/meshes/Battery---Battery-5.2-Ah-DC5521-Plug-v2.stl" scale="0.001 0.001 0.001" />
             </geometry>
+            <material name="battery_green"/>
         </visual>
         <collision name="Battery---Battery-5.2-Ah-DC5521-Plug-v2_collision">
@@ -319,4 +350,5 @@
                 <mesh filename="package://lekiwi_description/meshes/94868A713_NO-THREADS_Female-Threaded-Hex-Standoff.stl" scale="0.001 0.001 0.001" />
             </geometry>
+            <material name="silver"/>
         </visual>
         <collision name="94868A713_NO-THREADS_Female-Threaded-Hex-Standoff_collision">
@@ -338,4 +370,5 @@
                 <mesh filename="package://lekiwi_description/meshes/base_plate_layer2-v3.stl" scale="0.001 0.001 0.001" />
             </geometry>
+            <material name="base_dark_gray"/>
         </visual>
         <collision name="base_plate_layer2-v3_collision">
@@ -357,4 +390,5 @@
                 <mesh filename="package://lekiwi_description/meshes/Bottom-V2-v3.stl" scale="0.001 0.001 0.001" />
             </geometry>
+            <material name="arm_blue"/>
         </visual>
         <collision name="Bottom-V2-v3_collision">
@@ -376,4 +410,5 @@
                 <mesh filename="package://lekiwi_description/meshes/Top-V2-v2.stl" scale="0.001 0.001 0.001" />
             </geometry>
+            <material name="arm_blue"/>
         </visual>
         <collision name="Top-V2-v2_collision">
@@ -395,4 +430,5 @@
                 <mesh filename="package://lekiwi_description/meshes/Camera-Mount-v8.stl" scale="0.001 0.001 0.001" />
             </geometry>
+            <material name="cam_black"/>
         </visual>
         <collision name="Camera-Mount-v8_collision">
@@ -414,4 +450,5 @@
                 <mesh filename="package://lekiwi_description/meshes/Camera-Model-v3.stl" scale="0.001 0.001 0.001" />
             </geometry>
+            <material name="cam_black"/>
         </visual>
         <collision name="Camera-Model-v3_collision">
@@ -433,4 +470,5 @@
                 <mesh filename="package://lekiwi_description/meshes/Base_08q-v1.stl" scale="0.001 0.001 0.001" />
             </geometry>
+            <material name="arm_blue_dark"/>
         </visual>
         <collision name="Base_08q-v1_collision">
@@ -452,4 +490,5 @@
                 <mesh filename="package://lekiwi_description/meshes/WaveShare_Mounting_Plate_01d-v1.stl" scale="0.001 0.001 0.001" />
             </geometry>
+            <material name="pcb_green"/>
         </visual>
         <collision name="WaveShare_Mounting_Plate_01d-v1_collision">
@@ -471,4 +510,5 @@
                 <mesh filename="package://lekiwi_description/meshes/Rotation_Pitch_08i-v1.stl" scale="0.001 0.001 0.001" />
             </geometry>
+            <material name="arm_blue"/>
         </visual>
         <collision name="Rotation_Pitch_08i-v1_collision">
@@ -490,4 +530,5 @@
                 <mesh filename="package://lekiwi_description/meshes/STS3215_03a-v1.stl" scale="0.001 0.001 0.001" />
             </geometry>
+            <material name="arm_servo"/>
         </visual>
         <collision name="STS3215_03a-v1_collision">
@@ -509,4 +550,5 @@
                 <mesh filename="package://lekiwi_description/meshes/SO_ARM100_08k_Asym_Mirror_Clip-v1.stl" scale="0.001 0.001 0.001" />
             </geometry>
+            <material name="arm_blue"/>
         </visual>
         <collision name="SO_ARM100_08k_Asym_Mirror_Clip-v1_collision">
@@ -528,4 +570,5 @@
                 <mesh filename="package://lekiwi_description/meshes/Passive_Horn_01-v1.stl" scale="0.001 0.001 0.001" />
             </geometry>
+            <material name="gripper_teal"/>
         </visual>
         <collision name="Passive_Horn_01-v1_collision">
@@ -547,4 +590,5 @@
                 <mesh filename="package://lekiwi_description/meshes/STS3215_03a-v1-1.stl" scale="0.001 0.001 0.001" />
             </geometry>
+            <material name="arm_servo"/>
         </visual>
         <collision name="STS3215_03a-v1-1_collision">
@@ -566,4 +610,5 @@
                 <mesh filename="package://lekiwi_description/meshes/SO_ARM100_08k_116_Square-v1.stl" scale="0.001 0.001 0.001" />
             </geometry>
+            <material name="arm_blue"/>
         </visual>
         <collision name="SO_ARM100_08k_116_Square-v1_collision">
@@ -585,4 +630,5 @@
                 <mesh filename="package://lekiwi_description/meshes/STS3215_03a-v1-2.stl" scale="0.001 0.001 0.001" />
             </geometry>
+            <material name="arm_servo"/>
         </visual>
         <collision name="STS3215_03a-v1-2_collision">
@@ -604,4 +650,5 @@
                 <mesh filename="package://lekiwi_description/meshes/SO_ARM100_08k_Mirror-v1.stl" scale="0.001 0.001 0.001" />
             </geometry>
+            <material name="arm_blue"/>
         </visual>
         <collision name="SO_ARM100_08k_Mirror-v1_collision">
@@ -623,4 +670,5 @@
                 <mesh filename="package://lekiwi_description/meshes/STS3215_03a-v1-3.stl" scale="0.001 0.001 0.001" />
             </geometry>
+            <material name="arm_servo"/>
         </visual>
         <collision name="STS3215_03a-v1-3_collision">
@@ -642,4 +690,5 @@
                 <mesh filename="package://lekiwi_description/meshes/Wrist_Roll_Pitch_08i-v1.stl" scale="0.001 0.001 0.001" />
             </geometry>
+            <material name="arm_blue"/>
         </visual>
         <collision name="Wrist_Roll_Pitch_08i-v1_collision">
@@ -661,4 +710,5 @@
                 <mesh filename="package://lekiwi_description/meshes/STS3215_03a_Wrist_Roll-v1.stl" scale="0.001 0.001 0.001" />
             </geometry>
+            <material name="arm_servo"/>
         </visual>
         <collision name="STS3215_03a_Wrist_Roll-v1_collision">
@@ -680,4 +730,5 @@
                 <mesh filename="package://lekiwi_description/meshes/Wrist_Roll_08c-v1.stl" scale="0.001 0.001 0.001" />
             </geometry>
+            <material name="arm_blue"/>
         </visual>
         <collision name="Wrist_Roll_08c-v1_collision">
@@ -699,4 +750,5 @@
                 <mesh filename="package://lekiwi_description/meshes/STS3215_03a-v1-4.stl" scale="0.001 0.001 0.001" />
             </geometry>
+            <material name="arm_servo"/>
         </visual>
         <collision name="STS3215_03a-v1-4_collision">
@@ -718,4 +770,5 @@
                 <mesh filename="package://lekiwi_description/meshes/Moving_Jaw_08d-v1.stl" scale="0.001 0.001 0.001" />
             </geometry>
+            <material name="gripper_teal"/>
         </visual>
         <collision name="Moving_Jaw_08d-v1_collision">
@@ -737,4 +790,5 @@
                 <mesh filename="package://lekiwi_description/meshes/Wrist-Camera-Mount-v11.stl" scale="0.001 0.001 0.001" />
             </geometry>
+            <material name="cam_black"/>
         </visual>
         <collision name="Wrist-Camera-Mount-v11_collision">
@@ -756,4 +810,5 @@
                 <mesh filename="package://lekiwi_description/meshes/94868A713_NO-THREADS_Female-Threaded-Hex-Standoff-1.stl" scale="0.001 0.001 0.001" />
             </geometry>
+            <material name="silver"/>
         </visual>
         <collision name="94868A713_NO-THREADS_Female-Threaded-Hex-Standoff-1_collision">
@@ -775,4 +830,5 @@
                 <mesh filename="package://lekiwi_description/meshes/94868A713_NO-THREADS_Female-Threaded-Hex-Standoff-2.stl" scale="0.001 0.001 0.001" />
             </geometry>
+            <material name="silver"/>
         </visual>
         <collision name="94868A713_NO-THREADS_Female-Threaded-Hex-Standoff-2_collision">
@@ -794,4 +850,5 @@
                 <mesh filename="package://lekiwi_description/meshes/Camera-Model-v3-1.stl" scale="0.001 0.001 0.001" />
             </geometry>
+            <material name="cam_black"/>
         </visual>
         <collision name="Camera-Model-v3-1_collision">
@@ -813,4 +870,5 @@
                 <mesh filename="package://lekiwi_description/meshes/94868A713_NO-THREADS_Female-Threaded-Hex-Standoff-3.stl" scale="0.001 0.001 0.001" />
             </geometry>
+            <material name="silver"/>
         </visual>
         <collision name="94868A713_NO-THREADS_Female-Threaded-Hex-Standoff-3_collision">
@@ -832,4 +890,5 @@
                 <mesh filename="package://lekiwi_description/meshes/94868A713_NO-THREADS_Female-Threaded-Hex-Standoff-4.stl" scale="0.001 0.001 0.001" />
             </geometry>
+            <material name="silver"/>
         </visual>
         <collision name="94868A713_NO-THREADS_Female-Threaded-Hex-Standoff-4_collision">
@@ -851,4 +910,5 @@
                 <mesh filename="package://lekiwi_description/meshes/94868A713_NO-THREADS_Female-Threaded-Hex-Standoff-5.stl" scale="0.001 0.001 0.001" />
             </geometry>
+            <material name="silver"/>
         </visual>
         <collision name="94868A713_NO-THREADS_Female-Threaded-Hex-Standoff-5_collision">

Commit message: change wheel colision from sphere to cylinder

File: lekiwi_description/urdf/LeKiwi.xacro (robot description, xacro)
@@ -95,5 +95,5 @@
             <origin xyz="7.450578487500081e-12 0.015874999999999986 6.661338147750939e-18" rpy="1.5707963267948966 0.26179938779914924 -1.0046485565123013e-33" />
             <geometry>
-                <sphere radius="0.05" />
+                <cylinder radius="0.05" length="0.03"/>
             </geometry>
         </collision>
@@ -195,5 +195,5 @@
             <origin xyz="0.013748155931950041 -0.007937495502761073 -2.2204460492503132e-17" rpy="-0.5235987755982988 -1.5707963267948963 0" />
             <geometry>
-                <sphere radius="0.05" />
+                <cylinder radius="0.05" length="0.03"/>
             </geometry>
         </collision>
@@ -275,5 +275,5 @@
             <origin xyz="-0.013748155616372878 -0.007937504497239081 -5.773159728050814e-17" rpy="1.5707963267948974 -1.3089969389957468 2.094395102393195" />
             <geometry>
-                <sphere radius="0.05" />
+                <cylinder radius="0.05" length="0.03"/>
             </geometry>
         </collision>
@@ -920,5 +920,5 @@
     </link>
     <joint name="base_joint" type="fixed">
-        <origin xyz="0 0 0.025" rpy="0 0 0" />
+        <origin xyz="0 0 0.025" rpy="0 0 -${pi/2}" />
         <parent link="base_footprint" />
         <child link="base_plate_layer1-v5" />
