Commit message: update gz file

File: lekiwi_description/urdf/LeKiwi_gazebo.xacro (robot description, xacro)
@@ -1,5 +1,54 @@
 <?xml version="1.0"?>
 <robot xmlns:xacro="http://www.ros.org/wiki/xacro" xmlns:gz="http://gazebosim.org/schema">
-    <xacro:macro name="wheel_collision" params="wheel_link">
+    <!--
+    ════════════════════════════════════════════════════════════════
+      LeKiwi – Gazebo Harmonic friction / contact tuning
+    ════════════════════════════════════════════════════════════════
+    ROOT-CAUSE FIX (lateral motion random / robot rotates):
+    ─────────────────────────────────────────────────────────
+    fdir1 must point along the wheel's TANGENTIAL rolling direction,
+    NOT the radial direction.
+    ODE friction model at contact point:
+      • mu  (fdir1 axis)  = HIGH → the driven rolling direction.
+                                   Wheel rim grips ground here; motor
+                                   force propels the robot.
+      • mu2 (⊥ to fdir1) = LOW  → the passive-roller axis.
+                                   Small barrel rollers spin freely;
+                                   wheel slides sideways with no
+                                   motor resistance.
+    For a wheel at polar angle θ from robot origin (top view):
+      Radial direction     = ( sin θ,  cos θ, 0 )  ← v1 (was wrong)
+      Tangential direction = ( cos θ, -sin θ, 0 )  ← v2 (correct)
+    The three tangential vectors are 120° apart:
+      v1-2  θ = 0      →  ( 1.000,  0.000, 0 )
+      v1-1  θ = 2π/3  →  (-0.500, -0.866, 0 )
+      v1    θ = 4π/3  →  (-0.500,  0.866, 0 )
+    ── TUNABLE CONSTANTS ────────────────────────────────────────────
+    kp        Spring stiffness [N/m]. Raise if wheel sinks into
+              ground; lower if sim jitters. Sphere colliders need
+              lower values than cylinder/capsule.
+    kd        Damping [N·s/m].  Rule of thumb: kd ≈ kp × 0.01.
+    mu        Rolling-direction friction (HIGH).
+              Raise if wheel slips in commanded direction (max ~2.0).
+    mu2       Passive-roller-direction friction (LOW).
+              Lower → freer strafing.  Higher → stiffer lateral feel.
+    min_depth Contact depth threshold [m]. Prevents micro-jitter when
+              sphere barely grazes the ground plane.
+    max_vel   Max penetration-correction velocity [m/s]. Caps the
+              explosive impulse generated on first contact.
+    ════════════════════════════════════════════════════════════════
+    -->
+    <xacro:property name="wheel_kp"       value="2e5"   />
+    <xacro:property name="wheel_kd"       value="2e3"   />
+    <xacro:property name="wheel_mu"       value="1.2"   />
+    <xacro:property name="wheel_mu2"      value="0.05" />
+    <xacro:property name="wheel_minDepth" value="0.001" />
+    <xacro:property name="wheel_maxVel"   value="0.1"   />
+    <!-- ──────────────────────────────────────────────────────────
+         MACRO: applies per-wheel surface properties.
+         fdir1 expressed in base_footprint → stays fixed relative
+         to the robot body even as the wheel spins.
+         ────────────────────────────────────────────────────────── -->
+    <xacro:macro name="wheel_collision" params="wheel_link fdir1_x fdir1_y fdir1_z">
         <gazebo reference="${wheel_link}">
             <collision>
@@ -7,13 +56,17 @@
                     <contact>
                         <ode>
-                            <kp>1.5e6</kp>
-                            <kd>2e4</kd>
+                            <kp>${wheel_kp}</kp>
+                            <kd>${wheel_kd}</kd>
+                            <min_depth>${wheel_minDepth}</min_depth>
+                            <max_vel>${wheel_maxVel}</max_vel>
                         </ode>
                     </contact>
                     <friction>
                         <ode>
-                            <mu>0.6</mu>
-                            <mu2>0.1</mu2>
-                            <fdir1 gz:expressed_in="base_footprint">1 0 0</fdir1>
+                            <!-- HIGH friction → driven rolling direction -->
+                            <mu>${wheel_mu}</mu>
+                            <!-- LOW  friction → passive roller direction  -->
+                            <mu2>${wheel_mu2}</mu2>
+                            <fdir1 gz:expressed_in="base_footprint">${fdir1_x} ${fdir1_y} ${fdir1_z}</fdir1>
                         </ode>
                     </friction>
@@ -22,18 +75,40 @@
         </gazebo>
     </xacro:macro>
-    <xacro:wheel_collision wheel_link="4-Omni-Directional-Wheel_Single_Body-v1-1" />
-    <xacro:wheel_collision wheel_link="4-Omni-Directional-Wheel_Single_Body-v1-2" />
-    <xacro:wheel_collision wheel_link="4-Omni-Directional-Wheel_Single_Body-v1" />
+    <!-- ──────────────────────────────────────────────────────────
+         WHEEL INSTANCES
+         Formula: fdir1 = ( cos(θ), -sin(θ), 0 )  ← tangential
+         ────────────────────────────────────────────────────────── -->
+    <!-- Wheel 0  θ = 0       fdir1 = ( 1.000,  0.000, 0 ) -->
+    <xacro:wheel_collision
+        wheel_link="4-Omni-Directional-Wheel_Single_Body-v1-2"
+        fdir1_x="${cos(0)}"
+        fdir1_y="${-sin(0)}"
+        fdir1_z="0" />
+    <!-- Wheel 1  θ = 2π/3   fdir1 = (-0.500, -0.866, 0 ) -->
+    <xacro:wheel_collision
+        wheel_link="4-Omni-Directional-Wheel_Single_Body-v1-1"
+        fdir1_x="${cos(2*pi/3)}"
+        fdir1_y="${-sin(2*pi/3)}"
+        fdir1_z="0" />
+    <!-- Wheel 2  θ = 4π/3   fdir1 = (-0.500,  0.866, 0 ) -->
+    <xacro:wheel_collision
+        wheel_link="4-Omni-Directional-Wheel_Single_Body-v1"
+        fdir1_x="${cos(4*pi/3)}"
+        fdir1_y="${-sin(4*pi/3)}"
+        fdir1_z="0" />
+    <!-- ──────────────────────────────────────────────────────────
+         PLUGINS
+         ────────────────────────────────────────────────────────── -->
     <gazebo>
         <plugin filename="gz-sim-imu-system" name="gz::sim::systems::Imu">
-      </plugin>
+        </plugin>
     </gazebo>
     <gazebo>
-      <plugin filename="gz-sim-sensors-system" name="gz::sim::systems::Sensors">
-        <render_engine>ogre2</render_engine>
-      </plugin>
-      <plugin filename="gz_ros2_control-system" name="gz_ros2_control::GazeboSimROS2ControlPlugin">
-        <parameters>$(find lekiwi_controller)/config/lekiwi_controllers.yaml</parameters>
-      </plugin>
+        <plugin filename="gz-sim-sensors-system" name="gz::sim::systems::Sensors">
+            <render_engine>ogre2</render_engine>
+        </plugin>
+        <plugin filename="gz_ros2_control-system" name="gz_ros2_control::GazeboSimROS2ControlPlugin">
+            <parameters>$(find lekiwi_controller)/config/lekiwi_controllers.yaml</parameters>
+        </plugin>
     </gazebo>
 </robot>
